Commit message: first working passive simulation with mobile base only

File: drake/examples/TRI_Remy/remy_description/robot/remy.urdf (robot description, URDF)
Before this commit: robot remy_description, 4 links, 3 joints
Links:
- added link back_caster_mount, mass 0.107381888645876; collision mesh filename=../meshes/back_caster_mount.obj; visual mesh filename=../meshes/back_caster_mount.obj
- added link back_caster_wheel, mass 0.185602296468908; collision mesh filename=../meshes/back_caster_wheel.obj; visual mesh filename=../meshes/back_caster_wheel.obj
- added link front_caster_mount, mass 0.107382154839307; collision mesh filename=../meshes/front_caster_mount.obj; visual mesh filename=../meshes/front_caster_mount.obj
- added link front_caster_wheel, mass 0.185602296468908; collision mesh filename=../meshes/front_caster_wheel.obj; visual mesh filename=../meshes/front_caster_wheel.obj
- added link jaco_mount, mass 0.12648183952591; collision mesh filename=../meshes/jaco_mount.obj; visual mesh filename=../meshes/jaco_mount.obj
- link base_link: mass 3.7861195695851 -> 8.46822252536056
- link lift: mass 1.10311860062385 -> 1.10311806702314
Joints:
- added joint back_caster: type continuous, parent base_link, child back_caster_mount, origin xyz=0 0.2286 -0.00331958737700475 rpy=0.0523598775586215 -5.92206520112322E-17 -1.82771088172709, axis 0 0.0523359562417371 0.998629534754637
- added joint back_caster_wheel: type continuous, parent back_caster_mount, child back_caster_wheel, origin xyz=0 0.0294020016398932 -0.0759667553055578 rpy=1.5707963267949 -0.616507014374687 -1.5707963267949, axis 0 0 -1
- added joint front_caster: type continuous, parent base_link, child front_caster_mount, origin xyz=0 -0.2286 -0.0033196 rpy=0.05236 -2.0274E-17 -0.33749, axis 0 0.052336 0.99863
- added joint front_caster_wheel: type continuous, parent front_caster_mount, child front_caster_wheel, origin xyz=0 0.0294020016396793 -0.0759667553056439 rpy=1.5707963267949 -0.616507014377602 -1.57079632679489, axis 0 0 -1
- added joint jaco_mount: type fixed, parent lift, child jaco_mount, origin xyz=0.0173989999999999 0.159412958043339 0.00572157209564689 rpy=0.261799387799146 8.34582944186186E-17 -3.14159265358979, axis 0 0 0
- joint lift: origin xyz=0.017399 -0.033223 0.11124 rpy=0.2618 1.0643E-16 -3.1416 -> xyz=0.017399 -0.040484 0.084147 rpy=0.2618 1.0643E-16 -3.1416

Commit message: Removed all collision elements except wheels. Added friction parameters to demo

File: drake/examples/TRI_Remy/remy_description/robot/remy.urdf (robot description, URDF)
Before this commit: robot remy_description, 9 links, 8 joints
Links:
- link back_caster_mount: geometry visual mesh filename=../meshes/back_caster_mount.obj
- link base_link: geometry visual mesh filename=../meshes/base_link.obj
- link front_caster_mount: geometry visual mesh filename=../meshes/front_caster_mount.obj
- link jaco_mount: geometry visual mesh filename=../meshes/jaco_mount.obj
- link lift: geometry visual mesh filename=../meshes/lift.obj
Joints:
- joint lift: limit lower=0 upper=0.6 effort=0 velocity=0 -> lower=0.1 upper=0.6 effort=0 velocity=0

Commit message: Added kinova arm to MMB. First working simulation of full Remy

File: drake/examples/TRI_Remy/remy_description/robot/remy.urdf (robot description, URDF)
Before this commit: robot remy_description, 9 links, 8 joints
Links:
- added link j2n6s300_end_effector; collision box size=0 0 0; visual box size=0 0 0
- added link j2n6s300_link_1, mass 0.7477; collision cylinder length=0.06 radius=0.025; visual mesh filename=../../../../manipulation/models/jaco_description/meshes/rin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
- added link j2n6s300_link_2, mass 0.99; collision cylinder length=0.3 radius=0.025; visual mesh filename=../../../../manipulation/models/jaco_description/meshes/arm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
- added link j2n6s300_link_3, mass 0.6763; collision cylinder length=0.17 radius=0.025; visual mesh filename=../../../../manipulation/models/jaco_description/meshes/for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
- added link j2n6s300_link_4, mass 0.1785; collision cylinder length=0.01 radius=0.025; visual mesh filename=../../../../manipulation/models/jaco_description/meshes/rin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
- added link j2n6s300_link_5, mass 0.1785; collision cylinder length=0.01 radius=0.025; visual mesh filename=../../../../manipulation/models/jaco_description/meshes/rin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
- added link j2n6s300_link_6, mass 0.727; collision cylinder length=0.01 radius=0.025; visual mesh filename=../../../../manipulation/models/jaco_description/meshes/han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
- added link j2n6s300_link_base, mass 0.46784; collision cylinder length=0.075 radius=0.025; visual mesh filename=../../../../manipulation/models/jaco_description/meshes/bas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
- added link j2n6s300_link_finger_1, mass 0.01; collision cylinder length=0.01 radius=0.01; visual mesh filename=../../../../manipulation/models/jaco_description/meshes/fin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
- added link j2n6s300_link_finger_2, mass 0.01; collision cylinder length=0.01 radius=0.01; visual mesh filename=../../../../manipulation/models/jaco_description/meshes/fin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
- added link j2n6s300_link_finger_3, mass 0.01; collision cylinder length=0.01 radius=0.01; visual mesh filename=../../../../manipulation/models/jaco_description/meshes/fin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
- added link j2n6s300_link_finger_tip_1, mass 0.01; collision cylinder length=0.01 radius=0.01; visual mesh filename=../../../../manipulation/models/jaco_description/meshes/fin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
- added link j2n6s300_link_finger_tip_2, mass 0.01; collision cylinder length=0.01 radius=0.01; visual mesh filename=../../../../manipulation/models/jaco_description/meshes/fin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
- added link j2n6s300_link_finger_tip_3, mass 0.01; collision cylinder length=0.01 radius=0.01; visual mesh filename=../../../../manipulation/models/jaco_description/meshes/fin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
Joints:
- added joint j2n6s300_joint_1: type continuous, parent j2n6s300_link_base, child j2n6s300_link_1, origin xyz=0 0 0.15675 rpy=0 3.14159265359 0, axis 0 0 1, limit lower=-6.28318530718 upper=6.28318530718 effort=2000 velocity=1
- added joint j2n6s300_joint_2: type fixed, parent j2n6s300_link_1, child j2n6s300_link_2, origin xyz=0 0.0016 -0.11875 rpy=-1.57079632679 -1.57 3.14159265359, axis 0 0 1, limit lower=-2.618 upper=2.613 effort=2000 velocity=1
- added joint j2n6s300_joint_3: type revolute, parent j2n6s300_link_2, child j2n6s300_link_3, origin xyz=0 -0.410 0 rpy=0 3.14159265359 3.1415, axis 0 0 1, limit lower=-2.618 upper=2.613 effort=2000 velocity=1
- added joint j2n6s300_joint_4: type continuous, parent j2n6s300_link_3, child j2n6s300_link_4, origin xyz=0 0.2073 -0.0114 rpy=-1.57079632679 0 3.14159265359, axis 0 0 1, limit lower=-6.28318530718 upper=6.28318530718 effort=2000 velocity=1
- added joint j2n6s300_joint_5: type continuous, parent j2n6s300_link_4, child j2n6s300_link_5, origin xyz=0 -0.03703 -0.06414 rpy=1.0471975512 0 3.14159265359, axis 0 0 1, limit lower=-6.28318530718 upper=6.28318530718 effort=2000 velocity=1
- added joint j2n6s300_joint_6: type continuous, parent j2n6s300_link_5, child j2n6s300_link_6, origin xyz=0 -0.03703 -0.06414 rpy=1.0471975512 0 3.14159265359, axis 0 0 1, limit lower=-6.28318530718 upper=6.28318530718 effort=2000 velocity=1
- added joint j2n6s300_joint_base: type fixed, parent jaco_mount, child j2n6s300_link_base, origin xyz=0 0 0 rpy=0 0 0, axis 0 0 0, limit lower=0 upper=0 effort=2000 velocity=1
- added joint j2n6s300_joint_end_effector: type fixed, parent j2n6s300_link_6, child j2n6s300_end_effector, origin xyz=0 0 -0.1600 rpy=3.14159265359 0 0, axis 0 0 0, limit lower=0 upper=0 effort=2000 velocity=1
- added joint j2n6s300_joint_finger_1: type revolute, parent j2n6s300_link_6, child j2n6s300_link_finger_1, origin xyz=0.00279 0.03126 -0.11467 rpy=-1.570796327 .649262481663582 1.35961148639407, axis 0 0 1, limit lower=0 upper=2 effort=2000 velocity=1
- added joint j2n6s300_joint_finger_2: type revolute, parent j2n6s300_link_6, child j2n6s300_link_finger_2, origin xyz=0.02226 -0.02707 -0.11482 rpy=-1.570796327 .649262481663582 -1.38614049188413, axis 0 0 1, limit lower=0 upper=2 effort=2000 velocity=1
- added joint j2n6s300_joint_finger_3: type revolute, parent j2n6s300_link_6, child j2n6s300_link_finger_3, origin xyz=-0.02226 -0.02707 -0.11482 rpy=-1.570796327 .649262481663582 -1.75545216211587, axis 0 0 1, limit lower=0 upper=2 effort=2000 velocity=1
- added joint j2n6s300_joint_finger_tip_1: type fixed, parent j2n6s300_link_finger_1, child j2n6s300_link_finger_tip_1, origin xyz=0.044 -0.003 0 rpy=0 0 0, axis 0 0 1, limit lower=0 upper=2 effort=2000 velocity=1
- added joint j2n6s300_joint_finger_tip_2: type fixed, parent j2n6s300_link_finger_2, child j2n6s300_link_finger_tip_2, origin xyz=0.044 -0.003 0 rpy=0 0 0, axis 0 0 1, limit lower=0 upper=2 effort=2000 velocity=1
- added joint j2n6s300_joint_finger_tip_3: type fixed, parent j2n6s300_link_finger_3, child j2n6s300_link_finger_tip_3, origin xyz=0.044 -0.003 0 rpy=0 0 0, axis 0 0 1, limit lower=0 upper=2 effort=2000 velocity=1
- joint lift: limit lower=0.1 upper=0.6 effort=0 velocity=0 -> lower=0.7 upper=1 effort=0 velocity=0
