Commit message: updated keyframes, models, and added tables to sim. Also cleaned up directory.

File: drake/manipulation/models/iiwa_description/urdf/dual_iiwa14_primitive_sphere_collision_only.urdf (robot description, URDF)
Before this commit: robot dual_iiwa14, 21 links, 20 joints
Links:
- link left_iiwa_link_7: geometry collision mesh filename=../meshes/collision/link_7_polytope.obj; visual mesh filename=../meshes/collision/link_7_polytope.obj
- link right_iiwa_link_7: geometry collision mesh filename=../meshes/collision/link_7_polytope.obj; visual mesh filename=../meshes/collision/link_7_polytope.obj

File: drake/manipulation/models/iiwa_description/urdf/dual_iiwa14_primitive_sphere_visual_collision.urdf (robot description, URDF)
Before this commit: robot dual_iiwa14, 21 links, 20 joints
Links:
- link left_iiwa_link_7: geometry collision mesh filename=../meshes/collision/link_7_polytope.obj; visual mesh filename=../meshes/collision/link_7_polytope.obj
- link right_iiwa_link_7: geometry collision mesh filename=../meshes/collision/link_7_polytope.obj; visual mesh filename=../meshes/collision/link_7_polytope.obj
