Commit message: adding contact viz

File: drake/examples/kuka_iiwa_arm/dev/box_rotation/box.urdf (robot description, URDF)
Before this commit: robot box, 1 links, 0 joints
Links:
- link box: geometry collision box size=0.56 0.56 0.4; collision sphere radius=1e-2

Commit message: Working version of box rotation demo

File: drake/examples/kuka_iiwa_arm/dev/box_rotation/box.urdf (robot description, URDF)
Before this commit: robot box, 1 links, 0 joints
Links:
- link box: mass 1 -> 1.27; geometry collision box size=0.56 0.56 0.56; collision sphere radius=1e-3
