Commit message: shifted inner arm distance to match real iiwa's (after bolting down). Adjusted key frames slightly to work with new positions

File: examples/kuka_iiwa_arm/dev/box_rotation/models/dual_iiwa14_primitive_sphere_visual_collision.urdf (robot description, URDF)
Before this commit: robot dual_iiwa14, 21 links, 20 joints
Joints:
- joint left_iiwa_base_joint: origin xyz=0 0.9 0 rpy=0 0 0 -> xyz=0 0.8746 0 rpy=0 0 0
