Commit message: Adding actual kitchen models from Allison's CAD folder

File: examples/kuka_iiwa_arm/dev/box_rotation/models/hobart_rough.urdf (robot description, URDF)
Before this commit: robot hobart_rough, 4 links, 3 joints
Links:
- removed link bar
- removed link floor_pieces
- removed link lower_cabinet
- removed link upper_cabinet
- added link dishwasher_body; visual mesh filename=hobart_washer.obj scale=0.0254 0.0254 0.0254
Joints:
- removed joint floor_lower_joint
- removed joint lower_bar_joint
- removed joint lower_upper_joint

File: manipulation/models/iiwa_description/urdf/iiwa14_polytope_collision.urdf (robot description, URDF)
Before this commit: robot iiwa14, 11 links, 10 joints
Links:
- link iiwa_link_2: geometry visual mesh filename=../meshes/visual/link_2.obj; visual sphere radius=0.41
