Commit message: WIP for debugging anzu iiwa mug sim performance

File: manipulation/models/iiwa_description/urdf/iiwa14_polytope_collision.urdf (robot description, URDF)
Before this commit: robot iiwa14, 11 links, 10 joints
Links:
- link iiwa_link_7: geometry visual mesh filename=../meshes/visual/link_7.obj
