Commit message: Some fixes to support the teleop simulations in Rick's Anzu branch.

File: manipulation/models/iiwa_description/urdf/iiwa14_spheres_dense_elbow_collision.urdf (robot description, URDF)
Before this commit: robot iiwa14, 11 links, 10 joints
Links:
- link iiwa_link_7: geometry collision sphere radius=0.043; visual mesh filename=../meshes/visual/link_7.obj
