Commit message: Adds a planar-gripper simulation for brick rotation. Also adds QP and force control components.

File: examples/planar_gripper/planar_finger.xacro (robot description, xacro)
@@ -2,6 +2,6 @@
 <sdf xmlns:xacro="http://www.ros.org/wiki/xacro" version='1.6'>
   <model name='planar_gripper'>
-    <!-- Link mass and inertia values are guesses (currently), calculated using
-         a uniform rod model, rotating about its center of mass. -->
+    <!-- Link mass and inertia values are guessed, calculated using a
+         uniform rod model, rotating about its center of mass. -->
     <xacro:property name="base_dim" value=".08" />
     <xacro:property name="l1_length" value="0.085" />
@@ -13,8 +13,5 @@
     <xacro:property name="l1_zz_inertia" value="0.0006529" />
     <xacro:property name="l1_xz_inertia" value="0.000028883" />
-    <xacro:property name="l1_xy_inertia" value="0" />
-    <xacro:property name="l1_yz_inertia" value="0" />
     <xacro:property name="l2_length" value="0.040" />
-    <xacro:property name="l2_COM" value="0.02966" />
     <xacro:property name="l2_radius" value="0.011" />
     <xacro:property name="l2_mass" value="0.104" />
@@ -23,8 +20,6 @@
     <xacro:property name="l2_zz_inertia" value="0.000012773" />
     <xacro:property name="l2_xz_inertia" value="0.000006523" />
-    <xacro:property name="l2_xy_inertia" value="0" />
-    <xacro:property name="l2_yz_inertia" value="0" />
     <xacro:property name="shaft_inertia" value="0.0006" />
-    <xacro:property name="N" value="50" />  <!-- gear reduction -->
+    <xacro:property name="N" value="50" />
     <xacro:property name="sensor_length" value="0.005" />
     <xacro:property name="sensor_width" value="0.02" />
@@ -34,8 +29,4 @@
     <xacro:property name="tip_cylinder_radius" value="0.01" />
     <xacro:property name="tip_sphere_radius" value="0.015" />
-    <xacro:property name="base_joint_limit" value="1.570796" />
-    <xacro:property name="mid_joint_limit" value="1.570796" />
-    <xacro:property name="base_joint_damping" value="0" />
-    <xacro:property name="mid_joint_damping" value="0" />
     <xacro:macro name="finger" params="fnum">
       <link name="finger${fnum}_base">
@@ -55,20 +46,13 @@
         <pose>0 0 0 0 0 0</pose>
         <inertial>
-          <pose>0 0 -${l1_COM} 0 0 0</pose>
+          <pose>0 0 -${l1_length/2} 0 0 0</pose>
           <mass>${l1_mass}</mass>
           <inertia>
-            <!-- This includes the inertia contributed by the motor shaft
-                through the gear ratio N, shifted to the COM.
-                See planar_gripper.xacro for the calculation. Note that in
-                reality this inertia affects Ixx only, but we repeat the
-                calculation in Iyy and Izz to satisfy the triangle inequality.
-                This is really a hack for this special 2D case. In 3D, we would
-                have to model the motor shaft and gear reduction. -->
-            <ixx>${l1_xx_inertia + (shaft_inertia * N * N) + (l1_mass * l1_COM)}</ixx>
-            <iyy>${l1_yy_inertia + (shaft_inertia * N * N) + (l1_mass * l1_COM)}</iyy>
-            <izz>${l1_zz_inertia + (shaft_inertia * N * N) + (l1_mass * l1_COM)}</izz>
+            <ixx>${l1_xx_inertia + (shaft_inertia * N * N) + (l1_mass * l1_length/2)}</ixx>
+            <iyy>${l1_yy_inertia + (shaft_inertia * N * N) + (l1_mass * l1_length/2)}</iyy>
+            <izz>${l1_zz_inertia}</izz>
             <ixz>${l1_xz_inertia}</ixz>
-            <ixy>${l1_xy_inertia}</ixy>
-            <iyz>${l1_yz_inertia}</iyz>
+            <ixy>0</ixy>
+            <iyz>0</iyz>
           </inertia>
         </inertial>
@@ -104,10 +88,10 @@
           <limit>
             <!-- Drake parses a zero effort joint as an un-actuated joint. -->
-            <effort>75</effort>
-            <lower>-${base_joint_limit}</lower>
-            <upper>${base_joint_limit}</upper>
+            <effort>100</effort>
+            <lower>-2</lower>
+            <upper>2</upper>
           </limit>
           <dynamics>
-            <damping>${base_joint_damping}</damping>
+            <damping>0</damping>
           </dynamics>
           <use_parent_model_frame>1</use_parent_model_frame>
@@ -118,20 +102,13 @@
         <pose>0 0 -${l1_length} 0 0 0</pose>
         <inertial>
-          <pose>0 0 -${l2_COM} 0 0 0</pose>
+          <pose>0 0 -${(l2_length + sensor_length + tip_adapter_length + tip_cylinder_length)/2} 0 0 0</pose>
           <mass>${l2_mass}</mass>
           <inertia>
-            <!-- This includes the inertia contributed by the motor shaft
-                through the gear ratio N, shifted to the COM.
-                See planar_gripper.xacro for the calculation. Note that in
-                reality this inertia affects Ixx only, but we repeat the
-                calculation in Iyy and Izz to satisfy the triangle inequality.
-                This is really a hack for this special 2D case. In 3D, we would
-                have to model the motor shaft and gear reduction. -->
-            <ixx>${l2_xx_inertia  + (shaft_inertia * N * N) + (l2_mass * l2_COM)}</ixx>
-            <iyy>${l2_yy_inertia  + (shaft_inertia * N * N) + (l2_mass * l2_COM)}</iyy>
-            <izz>${l2_zz_inertia  + (shaft_inertia * N * N) + (l2_mass * l2_COM)}</izz>
+            <ixx>${l2_xx_inertia  + (shaft_inertia * N * N) + (l1_mass * (l2_length + sensor_length + tip_adapter_length + tip_cylinder_length)/2)}</ixx>
+            <iyy>${l2_yy_inertia  + (shaft_inertia * N * N) + (l1_mass * (l2_length + sensor_length + tip_adapter_length + tip_cylinder_length)/2)}</iyy>
+            <izz>${l2_zz_inertia}</izz>
             <ixz>${l2_xz_inertia}</ixz>
-            <ixy>${l2_xy_inertia}</ixy>
-            <iyz>${l2_yz_inertia}</iyz>
+            <ixy>0</ixy>
+            <iyz>0</iyz>
           </inertia>
         </inertial>
@@ -182,19 +159,14 @@
           <xyz>1 0 0</xyz>
           <limit>
-            <effort>75</effort>
-            <lower>-${mid_joint_limit}</lower>
-            <upper>${mid_joint_limit}</upper>
+            <effort>100</effort>
+            <lower>-2</lower>
+            <upper>2</upper>
           </limit>
           <dynamics>
-            <damping>${mid_joint_damping}</damping>
+            <damping>0</damping>
           </dynamics>
           <use_parent_model_frame>1</use_parent_model_frame>
         </axis>
       </joint>
-      <!-- The tip link's mass/inertia values are already included in link 2,
-           which welds to this link. Hence, the values here are set to be
-           (effectively) zero. Note: This fingertip link and its corresponding
-           weld joint allows us to sense forces via MBP's reaction forces
-           output port. -->
       <link name="finger${fnum}_tip_link">
         <pose>0 0 -${l1_length + l2_length + sensor_length} 0 0 0</pose>
@@ -239,5 +211,5 @@
           </geometry>
           <material>
-            <diffuse>1 1 1 1</diffuse>
+            <diffuse>1 1 1 0.4</diffuse>
           </material>
         </visual>
@@ -261,6 +233,4 @@
     </xacro:macro>
     <xacro:finger fnum="1" />
-    <xacro:finger fnum="2" />
-    <xacro:finger fnum="3" />
   </model>
 </sdf>

Commit message: Updated planar_finger.sdf to number the finger (e.g., finger1_BaseJoint).
Also updated a few methods to take in finger number as a parameter.

File: examples/planar_gripper/planar_finger.xacro (robot description, xacro)
@@ -30,5 +30,5 @@
     <xacro:property name="tip_sphere_radius" value="0.015" />
     <xacro:macro name="finger" params="fnum">
-      <link name="finger_base">
+      <link name="finger${fnum}_base">
         <visual name='base_visual'>
           <pose>0 0 0 0 0 0</pose>
@@ -43,5 +43,5 @@
         </visual>
       </link>
-      <link name="finger_link1">
+      <link name="finger${fnum}_link1">
         <pose>0 0 0 0 0 0</pose>
         <inertial>
@@ -81,7 +81,7 @@
         </visual>
       </link>
-      <joint name='finger_BaseJoint' type='revolute'>
-        <child>finger_link1</child>
-        <parent>finger_base</parent>
+      <joint name='finger${fnum}_BaseJoint' type='revolute'>
+        <child>finger${fnum}_link1</child>
+        <parent>finger${fnum}_base</parent>
         <axis>
           <xyz>1 0 0</xyz>
@@ -98,5 +98,5 @@
         </axis>
       </joint>
-      <link name="finger_link2">
+      <link name="finger${fnum}_link2">
         <!-- The origin of the link2 frame is located at the MidJoint. -->
         <pose>0 0 -${l1_length} 0 0 0</pose>
@@ -151,7 +151,7 @@
         </visual>
       </link>
-      <joint name='finger_MidJoint' type='revolute'>
-        <parent>finger_link1</parent>
-        <child>finger_link2</child>
+      <joint name='finger${fnum}_MidJoint' type='revolute'>
+        <parent>finger${fnum}_link1</parent>
+        <child>finger${fnum}_link2</child>
         <!-- Pose X_CJ of the joint frame J in the frame C of the child link -->
         <pose>0 0 0 0 0 0</pose>
@@ -169,5 +169,5 @@
         </axis>
       </joint>
-      <link name="finger_tip_link">
+      <link name="finger${fnum}_tip_link">
         <pose>0 0 -${l1_length + l2_length + sensor_length} 0 0 0</pose>
         <inertial>
@@ -226,7 +226,7 @@
         </collision>
       </link>
-      <joint name='finger_sensor_weldjoint' type='fixed'>
-        <parent>finger_link2</parent>
-        <child>finger_tip_link</child>
+      <joint name='finger${fnum}_sensor_weldjoint' type='fixed'>
+        <parent>finger${fnum}_link2</parent>
+        <child>finger${fnum}_tip_link</child>
         <pose>0 0 0 0 0 0</pose>
       </joint>
